Commit message: adding imu link in urdf

File: husky_customization/husky_custom_description/urdf/custom_description.urdf.xacro (robot description, xacro)
@@ -50,4 +50,25 @@
     <origin xyz="0.45 0 0" rpy="3.1415927 0 0" />
   </joint>
+  <!-- Insert imu -->
+  <link name="imu_link">
+    <visual>
+      <geometry>
+        <box size="0.022 0.025 0.005">
+      </geometry>
+      <material name="black">
+        <color rgba="0 0 0 1.0" />
+      </material>
+    </visual>
+    <collision>
+      <origin xyz="0 0 0" rpy="0 0 0" />
+      <geometry>
+        <box size="0.022 0.025 0.005">
+      </geometry>
+    </collision>
+  <joint name="imu_joint" type="fixed">
+    <parent link="base_link" />
+    <child link="imu_link" />
+    <origin xyz="0 0.035 0" rpy="3.1415927 0 0" />
+  </joint>
   <!-- Insert GPS Mount -->
   <link name="GPS_mount_link">

Commit message: fixed offset error for imu

File: husky_customization/husky_custom_description/urdf/custom_description.urdf.xacro (robot description, xacro)
@@ -69,5 +69,5 @@
     <parent link="base_link" />
     <child link="imu_link" />
-    <origin xyz="0 0.035 0" rpy="3.1415927 0 0" />
+    <origin xyz="0 0.170 0" rpy="3.1415927 0 0" />
   </joint>
   <!-- Insert GPS Mount -->

Commit message: configuring imu

File: husky_customization/husky_custom_description/urdf/custom_description.urdf.xacro (robot description, xacro)
@@ -49,25 +49,4 @@
     <origin xyz="0.45 0 0" rpy="3.1415927 0 0" />
   </joint>
-  <!-- Insert imu -->
-  <link name="imu_link">
-    <visual>
-      <geometry>
-        <box size="0.022 0.025 0.005">
-      </geometry>
-      <material name="black">
-        <color rgba="0 0 0 1.0" />
-      </material>
-    </visual>
-    <collision>
-      <origin xyz="0 0 0" rpy="0 0 0" />
-      <geometry>
-        <box size="0.022 0.025 0.005">
-      </geometry>
-    </collision>
-  <joint name="imu_joint" type="fixed">
-    <parent link="base_link" />
-    <child link="imu_link" />
-    <origin xyz="0 0.170 0" rpy="3.1415927 0 0" />
-  </joint>
   <!-- Insert GPS Mount -->
   <link name="GPS_mount_link">

Commit message: adding range filter and move up laser in urdf

File: husky_customization/husky_custom_description/urdf/custom_description.urdf.xacro (robot description, xacro)
@@ -47,5 +47,5 @@
     <parent link="base_link" />
     <child link="laser_link" />
-    <origin xyz="0.45 0 0" rpy="3.1415927 0 0" />
+    <origin xyz="0.45 0.0 0.08" rpy="3.1415927 0 0" />
   </joint>
   <!-- Insert GPS Mount -->
